File: 5v-power-supply.sch (KiCad schematic (older format))
At the start: 35 parts, among them P7 CONN_01X03, Q5 Q_NPN_BEC, U4 LNK4023D, U6 EPC1716D

Commit message: sync.sh update
Parts:
- removed P?: CONN_01X03, symbol CONN_01X03
- added P3, P4: CONN_01X02, footprints:pheonix-connector-01x02-5mm, symbol CONN_01X02
Connections:
- net HV+: now also P3.1 (P1), P3.2 (P2)
- net HV-: now also P4.1 (P1)
- net RELAY: now also P4.2 (P2)
Other:
- moved on the sheet: P7
