File: 5v-power-supply.kicad_pcb (KiCad board)
At the start: 2 copper layers, 54.7 x 41.2 mm, 41 parts, among them P3 CONN_01X02, P4 CONN_01X02, P7 CONN_01X03, Q3 Q_NPN_BEC, Q5 Q_NPN_BEC, U4 LNK4023D, U6 EPC1716D

Commit message: sync.sh update
Parts:
- L2: footprint Capacitors_ThroughHole:C_Radial_D10_L13_P5 -> footprints:Inductor_Radial
- moved L2 13.7 mm to (100.5, 94.9)
- moved P3 13.5 mm to (90.2, 107.8), turned to 90 degrees
- moved C3 9.11 mm to (93.9, 97.7), turned to 90 degrees
- moved BR1 8.44 mm to (98.9, 100.7), turned to 0 degrees
- moved C8 1.43 mm to (112.5, 97.8), turned to 90 degrees
- moved RT1 1.02 mm to (91.4, 115.7)
- moved P4 0.05 mm to (89.8, 122.3)
Routing:
- net Net-(C12-Pad2): track 35.8 -> 45.6 mm, vias 0 -> 1
- net Net-(BR1-Pad1): track 22.5 -> 12.8 mm
- net HV+: track 4.68 -> 14.3 mm
- net Net-(C8-Pad2): track 12.8 -> 15.8 mm
- net Net-(BR1-Pad2): track 21.8 -> 24.7 mm
- net Net-(Q5-Pad1): track 13.9 -> 12.2 mm, vias 3 -> 2
- removed copper zone on B.Cu, net HV+
